File: Prometheus.kicad_pcb (KiCad board)
At the start: 2 copper layers, 78.1 x 46.3 mm, 22 parts, among them J1 PORTD Termianls, J2 Power Terminals, J3 PORTC Terminals, J4 PORTB 01x06 Terminals, J5 02x05 Pin_Header, J6 Power Jack-P9, J7 Power KRE, SW1 RST Push Button, U1 ATmega328-P, U2 LM7805 TO220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

Commit message: Updates
Parts:
- added C7: 100n 16V, Capacitor_THT:C_Disc_D4.7mm_W2.5mm_P5.00mm, F.Cu at (161.2, 84.9)
- added D3: 1N4007, Diode_THT:D_DO-41_SOD81_P10.16mm_Horizontal, F.Cu at (124.8, 90.5)
- J5: footprint Connector_PinSocket_2.54mm:PinSocket_2x05_P2.54mm_Vertical -> Connector_IDC:IDC-Header_2x05_P2.54mm_Vertical
- SW1: footprint Button_Switch_THT:SW_Tactile_Straight_KSA0Axx1LFTR -> Button_Switch_THT:SW_PUSH_6mm_H4.3mm
- moved C6 33.3 mm to (158.1, 84.9), turned to 90 degrees
- moved D2 24.0 mm to (135.4, 75.7)
- moved R3 9.59 mm to (152.4, 75.7)
- moved J5 2.79 mm to (185.3, 91.0)
- moved SW1 1.81 mm to (130.9, 97.1)
- moved C3 1.14 mm to (118.8, 85.4)
Connections:
- net /MISO renamed GPIO_PB4
- net /MOSI renamed GPIO_PB3
- net /PB0 renamed GPIO_PB0
- net /PB1 renamed GPIO_PB1
- net /PB2 renamed GPIO_PB2
- net /RST renamed GPIO_RST
- net /SCK renamed GPIO_PB5
- net Net-(J1-Pin_1) renamed GPIO_PD0
- net Net-(J1-Pin_2) renamed GPIO_PD1
- net Net-(J1-Pin_3) renamed GPIO_PD2
- net Net-(J1-Pin_4) renamed GPIO_PD3
- net Net-(J1-Pin_5) renamed GPIO_PD4
- net Net-(J1-Pin_6) renamed GPIO_PD5
- net Net-(J1-Pin_7) renamed GPIO_PD6
- net Net-(J1-Pin_8) renamed GPIO_PD7
- net Net-(J3-Pin_1) renamed GPIO_PC5
- net Net-(J3-Pin_2) renamed GPIO_PC4
- net Net-(J3-Pin_3) renamed GPIO_PC3
- net Net-(J3-Pin_4) renamed GPIO_PC2
- net Net-(J3-Pin_5) renamed GPIO_PC1
- net Net-(J3-Pin_6) renamed GPIO_PC0
- C3 pad 1: VCC -> VCC_D_REG
- C6 pad 1: VCC -> Net-(U1-AREF)
- U1 pad 21: +5V -> Net-(U1-AREF)
- U2 pad 1: VCC -> VCC_D_REG
Routing:
- net GPIO_PB5: track 40.7 -> 57.4 mm, vias 2 -> 0
- net GND: track 5.40 -> 19.3 mm, vias 2 -> 4
- net VCC: track 86.0 -> 74.4 mm
- net VCC_D_REG: track 0.00 -> 11.5 mm
- net GPIO_PB4: track 25.3 -> 31.2 mm
- net Net-(D2-A): track 12.1 -> 6.90 mm
- net GPIO_PD5: track 32.1 -> 35.9 mm
- net Net-(U1-AREF): track 0.00 -> 3.64 mm
- net GPIO_PD4: track 22.5 -> 25.7 mm
- net GPIO_PD6: track 29.7 -> 32.6 mm
- net GPIO_RST: track 96.8 -> 99.7 mm, vias 3 -> 2
- net GPIO_PD7: track 27.4 -> 29.7 mm
- net GPIO_PD3: track 20.9 -> 22.8 mm
- net GPIO_PB3: track 25.0 -> 26.8 mm
- net GPIO_PD2: track 18.6 -> 20.3 mm
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