File: Prometheus.kicad_sch (KiCad schematic)
At the start: 22 parts, among them J1 PORTD Termianls, J2 Power Terminals, J3 PORTC Terminals, J4 PORTB 01x06 Terminals, J5 02x05 Pin_Header, J6 Power Jack-P9, J7 Power KRE, SW1 RST Push Button, U1 ATmega328-P, U2 LM7805 TO220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

Commit message: Updates
Parts:
- added C7: 100n 16V, Capacitor_THT:C_Disc_D4.7mm_W2.5mm_P5.00mm, symbol Componentes:CAP 100n 16V
- added D3: 1N4007, Diode_THT:D_DO-41_SOD81_P10.16mm_Horizontal, symbol Componentes:D 1N4007 1A 1000V
- J5: footprint Connector_PinSocket_2.54mm:PinSocket_2x05_P2.54mm_Vertical -> Connector_IDC:IDC-Header_2x05_P2.54mm_Vertical
- SW1: footprint Button_Switch_THT:SW_Tactile_Straight_KSA0Axx1LFTR -> Button_Switch_THT:SW_PUSH_6mm_H4.3mm
Connections:
- net +5V: now also C7.1; no longer U1.21 (AREF)
- net GND: now also C7.2
- net VCC: now also D3.2 (A); no longer C3.1, C6.1, U2.1 (VI)
- net GPIO_PD5: now reaches J1.6 (Pin_6), U1.11 (PD5)
- net GPIO_PD6: now reaches J1.7 (Pin_7), U1.12 (PD6)
- net GPIO_PD7: now reaches J1.8 (Pin_8), U1.13 (PD7)
- net GPIO_PD0: now reaches J1.1 (Pin_1), U1.2 (PD0)
- net GPIO_PC0: now reaches J3.6 (Pin_6), U1.23 (PC0)
- net GPIO_PC1: now reaches J3.5 (Pin_5), U1.24 (PC1)
- net GPIO_PC2: now reaches J3.4 (Pin_4), U1.25 (PC2)
- net GPIO_PC3: now reaches J3.3 (Pin_3), U1.26 (PC3)
- net GPIO_PC4: now reaches J3.2 (Pin_2), U1.27 (PC4)
- net GPIO_PC5: now reaches J3.1 (Pin_1), U1.28 (PC5)
- net GPIO_PD1: now reaches J1.2 (Pin_2), U1.3 (PD1)
- net GPIO_PD2: now reaches J1.3 (Pin_3), U1.4 (PD2)
- net GPIO_PD3: now reaches J1.4 (Pin_4), U1.5 (PD3)
- net GPIO_PD4: now reaches J1.5 (Pin_5), U1.6 (PD4)
- net MISO renamed GPIO_PB4
- net MOSI renamed GPIO_PB3
- net PB0 renamed GPIO_PB0
- net PB1 renamed GPIO_PB1
- net PB2 renamed GPIO_PB2
- net RST renamed GPIO_RST
- net SCK renamed GPIO_PB5
- new net: C6.1, U1.21 (AREF)
- new net VCC_D_REG: C3.1, D3.1 (K), U2.1 (VI)
Other:
- note added: "ATmega328P - Circuito Básico do MCU"
- note added: "Alimentação"
- note added: "Barramentos de GPIOs - PORTx|B;C;D"
- note added: "Gravação ISP"
- note added: "LEDs indicadores"
- note added: "PB5 SINAL"
- note added: "POWER"
- title: Prometheus Devkit mk 1.0 -> Prometheus Devkit mk 1.1
- moved on the sheet: C1, C2, C3, C4, C5, D1, D2, J1, J2, J3, J4, J5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
